Commit message: Add sensor models and simulation launch files for polebot AMR
- Implemented camera, lidar, and ultrasonic sensor models in Xacro format.
- Created a simulation package with CMake configuration and launch files.
- Added world definition for testing in Gazebo, including various objects and a ground plane.
- Integrated sensor plugins for Gazebo simulation.
- Established a launch file to spawn the robot model and associated sensors in the simulation environment.
- Included necessary dependencies and licensing information in package.xml and LICENSE files.

File: src/polebot_amr_description/polebot_amr.urdf (robot description, URDF)
Before this commit: robot amr_robot, 4 links, 3 joints
Links:
- link chassis: geometry collision box size=1.15 0.7 1.4; visual mesh filename=package://polebot_amr_description/meshes/polebot_amr.stl scale=0.001 0.001 0.001
- link lidar_link: geometry collision mesh filename=package://polebot_amr_description/meshes/lidar.stl scale=0.001 0.001 0.001; visual mesh filename=package://polebot_amr_description/meshes/lidar.stl scale=0.001 0.001 0.001
- link ultrasonic_link: geometry collision box size=0.04 0.02 0.02; visual mesh filename=package://polebot_amr_description/meshes/hcsr04.stl scale=0.001 0.001 0.001

File: src/polebot_amr_description/urdf/meca/base.xacro (robot description, xacro)
@@ -1,5 +1,5 @@
 <?xml version="1.0"?>
 <robot xmlns:xacro="http://www.ros.org/wiki/xacro" name="robot">
-  <xacro:property name="mesh_path" value="$(find amr_description)/meshes"/>
+  <xacro:property name="mesh_path" value="$(find polebot_amr_description)/meshes"/>
   <link name="world"/> <!-- Frame racine ajoutée -->
   <link name="base_link"/>
@@ -13,5 +13,5 @@
       <origin xyz="0 0 0" rpy="0 0 0"/>
       <geometry>
-        <mesh filename="file://${mesh_path}/amr.stl" scale="0.001 0.001 0.001"/>
+        <mesh filename="file://${mesh_path}/polebot_amr.stl" scale="0.001 0.001 0.001"/>
       </geometry>
       <material name="gray">

File: src/polebot_amr_description/urdf/meca/wheel.xacro (robot description, xacro)
@@ -1,5 +1,5 @@
 <?xml version="1.0"?>
 <robot xmlns:xacro="http://www.ros.org/wiki/xacro" name="wheel">
-  <xacro:property name="mesh_path" value="$(find amr_description)/meshes"/>
+  <xacro:property name="mesh_path" value="$(find polebot_amr_description)/meshes"/>
   <xacro:macro name="wheel" params="
     name

File: src/polebot_amr_description/urdf/robot/main_robot.xacro (robot description, xacro)
@@ -2,10 +2,10 @@
 <robot xmlns:xacro="http://www.ros.org/wiki/xacro" xmlns:gz="http://gazebosim.org" name="main_robot">
   <!-- Inclusions des composants -->
-  <xacro:include filename="/home/amr/amr_ws/src/amr_description/urdf/meca/base.xacro"/>
-  <xacro:include filename="/home/amr/amr_ws/src/amr_description/urdf/meca/wheel.xacro"/>
-  <xacro:include filename="/home/amr/amr_ws/src/amr_description/urdf/sensors/ultrasonic_sensors.xacro"/>
-  <xacro:include filename="/home/amr/amr_ws/src/amr_description/urdf/sensors/lidar.xacro"/>
-  <xacro:include filename="/home/amr/amr_ws/src/amr_description/urdf/sensors/camera.xacro"/>
-  <xacro:include filename="/home/amr/amr_ws/src/amr_description/urdf/control/diff_drive.gazebo"/>
+  <xacro:include filename="/home/amr/polebot_amr_ws/src/polebot_amr_description/urdf/meca/base.xacro"/>
+  <xacro:include filename="/home/amr/polebot_amr_ws/src/polebot_amr_description/urdf/meca/wheel.xacro"/>
+  <xacro:include filename="/home/amr/polebot_amr_ws/src/polebot_amr_description/urdf/sensors/ultrasonic_sensors.xacro"/>
+  <xacro:include filename="/home/amr/polebot_amr_ws/src/polebot_amr_description/urdf/sensors/lidar.xacro"/>
+  <xacro:include filename="/home/amr/polebot_amr_ws/src/polebot_amr_description/urdf/sensors/camera.xacro"/>
+  <xacro:include filename="/home/amr/polebot_amr_ws/src/polebot_amr_description/urdf/control/diff_drive.gazebo"/>
   <!-- Capteurs Ultrason -->
   <xacro:ultrasonic_sensor

File: src/polebot_amr_description/urdf/sensors/camera.xacro (robot description, xacro)
@@ -1,5 +1,5 @@
 <?xml version="1.0"?>
 <robot xmlns:xacro="http://www.ros.org/wiki/xacro" name="camera">
-  <xacro:property name="mesh_path" value="$(find amr_description)/meshes"/>
+  <xacro:property name="mesh_path" value="$(find polebot_amr_description)/meshes"/>
   <!-- Macro pour une caméra avec pose mesh configurable -->
   <xacro:macro name="camera_sensor" params="

File: src/polebot_amr_description/urdf/sensors/lidar.xacro (robot description, xacro)
@@ -1,5 +1,5 @@
 <?xml version="1.0"?>
 <robot xmlns:xacro="http://www.ros.org/wiki/xacro" name="lidar">
-  <xacro:property name="mesh_path" value="$(find amr_description)/meshes"/>
+  <xacro:property name="mesh_path" value="$(find polebot_amr_description)/meshes"/>
   <!-- Macro lidar avec visual et collision identiques -->
   <xacro:macro name="lidar_sensor" params="

File: src/polebot_amr_description/urdf/sensors/ultrasonic_sensors.xacro (robot description, xacro)
@@ -1,5 +1,5 @@
 <?xml version="1.0"?>
 <robot xmlns:xacro="http://www.ros.org/wiki/xacro" name="ultrasonic_sensors">
-  <xacro:property name="mesh_path" value="$(find amr_description)/meshes"/>
+  <xacro:property name="mesh_path" value="$(find polebot_amr_description)/meshes"/>
   <!-- Macro Xacro pour un capteur ultrasonique avec position locale -->
   <xacro:macro name="ultrasonic_sensor" params="
