Commit message: Refactor code structure for improved readability and maintainability

File: src/polebot_amr_description/urdf/robot/main_robot.xacro (robot description, xacro)
@@ -35,5 +35,5 @@
     mesh="lidar.stl"/>
   <!-- Caméra -->
-  <xacro:camera_sensor
+  <!-- <xacro:camera_sensor
     name="camera_left"
     parent_link="chassis"
@@ -41,7 +41,7 @@
     joint_rpy="0 0 0.7854"
     mesh_xyz="0 0 0"
-    mesh_rpy="0 0 0"/>
+    mesh_rpy="0 0 0"/> -->
   <!-- Caméra -->
-  <xacro:camera_sensor
+  <!-- <xacro:camera_sensor
     name="camera_right"
     parent_link="chassis"
@@ -49,5 +49,11 @@
     joint_rpy="0 0 -0.7854"
     mesh_xyz="0 0 0"
-    mesh_rpy="0 0 0"/>
+    mesh_rpy="0 0 0"/> -->
+  <link name="camera_link"/>
+  <joint name="camera_joint" type="fixed">
+    <parent link="chassis"/>
+    <child link="camera_link"/>
+    <origin xyz="0.0 -0.492 0.12" rpy="0 0 0"/>
+  </joint>
   <!-- Wheel -->
   <xacro:wheel

Commit message: Fix URDF, SLAM launch, and fake odom publisher for improved robot simulation
Fix: Update URDF for sensor parent links and camera setup

The lidar and ultrasonic sensor parent links in the URDF were updated from "chassis" to "base_link". The camera setup was simplified by removing the left and right camera configuration and replacing it with a single camera.

Fix: Modify SLAM launch file

The `declare_sim_time_arg` was commented out in the SLAM launch file.

Fix: Improve fake odometry publisher

The timer period in the fake odometry publisher was reduced to 0.02 seconds. A check was added to skip updates if the time difference (dt) is too large, preventing jumps. The orientation values x and y were explicitly set to 0.0 in both the transform and odometry messages.
The dt value is now capped at a maximum of 0.1 to prevent large jumps.

Refactor: Update submodules to reflect dirty state

The submodules roboteq_ros2_driver, lsc_ros2_driver, and serial are updated to reflect their dirty state.

File: src/polebot_amr_description/urdf/robot/main_robot.xacro (robot description, xacro)
@@ -27,5 +27,5 @@
   <xacro:lidar_sensor
     name="lidar"
-    parent_link="chassis"
+    parent_link="base_link"
     joint_xyz="0.0 -0.492 0.272"
     joint_rpy="0 0 0"
@@ -35,16 +35,8 @@
   <!-- Caméra -->
   <xacro:camera_sensor
-    name="camera_left"
-    parent_link="chassis"
-    joint_xyz="0.24 -0.47 0.216"
-    joint_rpy="0 0 0.7854"
-    mesh_xyz="0 0 0"
-    mesh_rpy="0 0 0"/>
-  <!-- Caméra -->
-  <xacro:camera_sensor
-    name="camera_right"
-    parent_link="chassis"
-    joint_xyz="-0.24 -0.47 0.216"
-    joint_rpy="0 0 -0.7854"
+    name="camera"
+    parent_link="base_link"
+    joint_xyz="0.0 -0.47 0.216"
+    joint_rpy="0 0 0"
     mesh_xyz="0 0 0"
     mesh_rpy="0 0 0"/>

File: src/polebot_amr_description/urdf/sensors/ultrasonic_sensors.xacro (robot description, xacro)
@@ -43,5 +43,5 @@
     <!-- Joint fixe entre le capteur et le parent -->
     <joint name="${name}_joint" type="fixed">
-      <parent link="chassis"/>
+      <parent link="base_link"/>
       <child link="${name}"/>
       <origin xyz="${joint_xyz}" rpy="${joint_rpy}"/>
