Commit message: Refactor robot launch files and RViz configurations; add Orbbec camera integration and update URDF for improved robot model representation

File: src/polebot_amr_description/urdf/meca/base.xacro (robot description, xacro)
@@ -2,8 +2,8 @@
 <robot xmlns:xacro="http://www.ros.org/wiki/xacro" name="robot">
   <xacro:property name="mesh_path" value="$(find polebot_amr_description)/meshes"/>
-  <link name="world"/> <!-- Frame racine ajoutée -->
+  <link name="base_footprint"/>
   <link name="base_link"/>
-  <joint name="world_to_base" type="fixed"> <!-- Joint fixe vers base_link -->
-    <parent link="world"/>
+  <joint name="base_footprint_joint" type="fixed">
+    <parent link="base_footprint"/>
     <child link="base_link"/>
     <origin xyz="0 0 0" rpy="0 0 0"/>
@@ -20,16 +20,14 @@
     </visual>
     <collision>
-      <origin xyz="0 0 0.7" rpy="0 0 0"/>
+      <origin xyz="0 0 0.428" rpy="0 0 0"/>
       <geometry>
-        <box size="1.15 0.7 1.4"/>
+        <box size="0.7 1.15 0.7"/>
       </geometry>
     </collision>
     <inertial>
-      <origin xyz="0 0 0.7" rpy="0 0 0"/>
-      <mass value="100.0"/>
-      <inertia
-        ixx="10.0" ixy="0.0" ixz="0.0"
-        iyy="10.0" iyz="0.0"
-        izz="10.0"/>
+      <origin xyz="0 0 0.35" rpy="0 0 0"/>
+      <mass value="5.0"/> <!-- Poids réduit pour répartir avec roues -->
+      <!-- Inertie recalculée de manière approximative -->
+      <inertia ixx="0.41" ixy="0" ixz="0" iyy="0.755" iyz="0" izz="0.755"/>
     </inertial>
   </link>
@@ -39,3 +37,119 @@
     <origin xyz="0 0 0" rpy="0 0 0"/>
   </joint>
+  <link name="left_wheel">
+    <inertial>
+      <origin xyz="0 0 0" rpy="0 0 0"/>
+      <mass value="1.5"/> <!-- ↖ Plus lourd -->
+      <inertia
+        ixx="0.003" ixy="0.0" ixz="0.0"
+        iyy="0.003" iyz="0.0"
+        izz="0.002"/>
+    </inertial>
+    <collision>
+      <geometry>
+        <cylinder radius="0.07" length="0.05"/>
+      </geometry>
+      <origin xyz="0 0 0" rpy="0 0 0"/>
+      <surface>
+        <friction>
+          <ode>
+            <mu>1.0</mu>
+            <mu2>0.0</mu2>
+          </ode>
+        </friction>
+      </surface>
+    </collision>
+  </link>
+  <joint name="left_wheel_joint" type="continuous">
+    <parent link="chassis"/>
+    <child link="left_wheel"/>
+    <origin xyz="0.375 0.3 0.07" rpy="1.57 0 1.57"/> <!-- Position à adapter -->
+    <axis xyz="0 -1 0">
+        <dynamics damping="1.0" friction="0.5"/>  <!-- Ajout ici -->
+    </axis>
+  </joint>
+   <link name="right_wheel">
+    <inertial>
+      <origin xyz="0 0 0" rpy="0 0 0"/>
+      <mass value="1.5"/> <!-- ↖ Plus lourd -->
+      <inertia
+        ixx="0.003" ixy="0.0" ixz="0.0"
+        iyy="0.003" iyz="0.0"
+        izz="0.002"/>
+    </inertial>
+    <collision>
+      <geometry>
+        <cylinder radius="0.07" length="0.05"/>
+      </geometry>
+      <origin xyz="0 0 0" rpy="0 0 0"/>
+      <surface>
+        <friction>
+          <ode>
+            <mu>1.0</mu>
+            <mu2>0.0</mu2>
+          </ode>
+        </friction>
+      </surface>
+    </collision>
+  </link>
+  <joint name="right_wheel_joint" type="continuous">
+    <parent link="chassis"/>
+    <child link="right_wheel"/>
+    <origin xyz="-0.375 0.3 0.07" rpy="1.57 0 1.57"/> <!-- Position à adapter -->
+    <axis xyz="0 -1 0">
+        <dynamics damping="1.0" friction="0.5"/>  <!-- Ajout ici -->
+    </axis>
+  </joint>
+  <link name="front_left_caster">
+    <inertial>
+      <mass value="1.5"/>
+      <inertia ixx="0.41" ixy="0" ixz="0" iyy="0.755" iyz="0" izz="0.755"/>
+    </inertial>
+    <collision>
+      <geometry>
+        <cylinder radius="0.07" length="0.05"/>
+      </geometry>
+      <origin xyz="0 0 0" rpy="0 0 0"/>
+      <surface>
+        <friction>
+          <ode>
+            <mu>1.0</mu>
+            <mu2>0.0</mu2>
+          </ode>
+        </friction>
+      </surface>
+    </collision>
+  </link>
+  <joint name="front_left_caster_joint" type="continuous">
+    <parent link="chassis"/>
+    <child link="front_left_caster"/>
+    <origin xyz="0.375 -0.3 0.07" rpy="1.57 0 1.57"/> <!-- Position adaptée -->
+    <axis xyz="0 -1 0"/>
+  </joint>
+  <link name="front_right_caster">
+    <inertial>
+      <mass value="1.5"/>
+      <inertia ixx="0.41" ixy="0" ixz="0" iyy="0.755" iyz="0" izz="0.755"/>
+    </inertial>
+    <collision>
+      <geometry>
+        <cylinder radius="0.07" length="0.05"/>
+      </geometry>
+      <origin xyz="0 0 0" rpy="0 0 0"/>
+      <surface>
+        <friction>
+          <ode>
+            <mu>1.0</mu>
+            <mu2>0.0</mu2>
+          </ode>
+        </friction>
+      </surface>
+    </collision>
+  </link>
+  <joint name="front_right_caster_joint" type="continuous">
+    <parent link="chassis"/>
+    <child link="front_right_caster"/>
+    <origin xyz="-0.375 -0.3 0.07" rpy="1.57 0 1.57"/> <!-- Position adaptée -->
+    <axis xyz="0 -1 0"/>
+  </joint>
 </robot>

File: src/polebot_amr_description/urdf/robot/main_robot.xacro (robot description, xacro)
@@ -30,40 +30,14 @@
     parent_link="chassis"
     joint_xyz="0.0 -0.492 0.272"
-    joint_rpy="0 0 0"
+    joint_rpy="0 0 3.14"
     mesh_xyz="0 0 0"
     mesh_rpy="0 0 0"
     mesh="lidar.stl"/>
   <!-- Caméra -->
-  <!-- <xacro:camera_sensor
-    name="camera_left"
-    parent_link="chassis"
-    joint_xyz="0.24 -0.47 0.216"
-    joint_rpy="0 0 0.7854"
-    mesh_xyz="0 0 0"
-    mesh_rpy="0 0 0"/> -->
-  <!-- Caméra -->
-  <!-- <xacro:camera_sensor
-    name="camera_right"
-    parent_link="chassis"
-    joint_xyz="-0.24 -0.47 0.216"
-    joint_rpy="0 0 -0.7854"
-    mesh_xyz="0 0 0"
-    mesh_rpy="0 0 0"/> -->
   <link name="camera_link"/>
   <joint name="camera_joint" type="fixed">
     <parent link="chassis"/>
     <child link="camera_link"/>
-    <origin xyz="0.0 -0.492 0.12" rpy="0 0 0"/>
+    <origin xyz="0.0 -0.492 0.12" rpy="0 0 1.57"/>
   </joint>
-  <!-- Wheel -->
-  <xacro:wheel
-    name="left_wheel"
-    parent_link="chassis"
-    joint_xyz="0.34 -0.1 0"
-    joint_rpy="0 0 0"/>
-  <xacro:wheel
-    name="right_wheel"
-    parent_link="chassis"
-    joint_xyz="-0.34 -0.1 0"
-    joint_rpy="0 0 0"/>
 </robot>

Commit message: Update launch files, add joystick configuration, and modify URDF for improved robot model

File: src/polebot_amr_description/urdf/meca/base.xacro (robot description, xacro)
@@ -20,5 +20,5 @@
     </visual>
     <collision>
-      <origin xyz="0 0 0.428" rpy="0 0 0"/>
+      <origin xyz="0 0 0" rpy="0 0 0"/>
       <geometry>
         <box size="0.7 1.15 0.7"/>
@@ -62,5 +62,5 @@
   </link>
   <joint name="left_wheel_joint" type="continuous">
-    <parent link="chassis"/>
+    <parent link="base_link"/>
     <child link="left_wheel"/>
     <origin xyz="0.375 0.3 0.07" rpy="1.57 0 1.57"/> <!-- Position à adapter -->
@@ -94,5 +94,5 @@
   </link>
   <joint name="right_wheel_joint" type="continuous">
-    <parent link="chassis"/>
+    <parent link="base_link"/>
     <child link="right_wheel"/>
     <origin xyz="-0.375 0.3 0.07" rpy="1.57 0 1.57"/> <!-- Position à adapter -->
@@ -122,5 +122,5 @@
   </link>
   <joint name="front_left_caster_joint" type="continuous">
-    <parent link="chassis"/>
+    <parent link="base_link"/>
     <child link="front_left_caster"/>
     <origin xyz="0.375 -0.3 0.07" rpy="1.57 0 1.57"/> <!-- Position adaptée -->
@@ -148,5 +148,5 @@
   </link>
   <joint name="front_right_caster_joint" type="continuous">
-    <parent link="chassis"/>
+    <parent link="base_link"/>
     <child link="front_right_caster"/>
     <origin xyz="-0.375 -0.3 0.07" rpy="1.57 0 1.57"/> <!-- Position adaptée -->

File: src/polebot_amr_description/urdf/robot/main_robot.xacro (robot description, xacro)
@@ -8,5 +8,4 @@
   <xacro:include filename="/home/amr/polebot_amr_ws/src/polebot_amr_description/urdf/sensors/camera.xacro"/>
   <xacro:include filename="/home/amr/polebot_amr_ws/src/polebot_amr_description/urdf/control/diff_drive.gazebo"/>
-  <!-- Capteurs Ultrason -->
   <xacro:ultrasonic_sensor
     name="uls_frontleft"
@@ -30,14 +29,23 @@
     parent_link="chassis"
     joint_xyz="0.0 -0.492 0.272"
-    joint_rpy="0 0 3.14"
+    joint_rpy="0 0 0"
     mesh_xyz="0 0 0"
     mesh_rpy="0 0 0"
     mesh="lidar.stl"/>
   <!-- Caméra -->
-  <link name="camera_link"/>
-  <joint name="camera_joint" type="fixed">
-    <parent link="chassis"/>
-    <child link="camera_link"/>
-    <origin xyz="0.0 -0.492 0.12" rpy="0 0 1.57"/>
-  </joint>
+  <xacro:camera_sensor
+    name="camera_left"
+    parent_link="chassis"
+    joint_xyz="0.24 -0.47 0.216"
+    joint_rpy="0 0 0.7854"
+    mesh_xyz="0 0 0"
+    mesh_rpy="0 0 0"/>
+  <!-- Caméra -->
+  <xacro:camera_sensor
+    name="camera_right"
+    parent_link="chassis"
+    joint_xyz="-0.24 -0.47 0.216"
+    joint_rpy="0 0 -0.7854"
+    mesh_xyz="0 0 0"
+    mesh_rpy="0 0 0"/>
 </robot>

Commit message: update

File: src/polebot_amr_description/urdf/meca/base.xacro (robot description, xacro)
@@ -7,14 +7,14 @@
     <parent link="base_footprint"/>
     <child link="base_link"/>
-    <origin xyz="0 0 0" rpy="0 0 0"/>
+    <origin xyz="0 0 0" rpy="0 0 -1.57"/>
   </joint>
   <link name="chassis">
     <visual>
-      <origin xyz="0 0 0" rpy="0 0 0"/>
+      <origin xyz="0 0 0" rpy="0 0 1.57"/>
       <geometry>
         <mesh filename="file://${mesh_path}/polebot_amr.stl" scale="0.001 0.001 0.001"/>
       </geometry>
       <material name="gray">
-        <color rgba="0.6 0.6 0.6 1.0"/>
+        <color rgba="0.3 0.3 0.3 1.0"/>
       </material>
     </visual>

File: src/polebot_amr_description/urdf/robot/main_robot.xacro (robot description, xacro)
@@ -28,5 +28,5 @@
     name="lidar"
     parent_link="base_link"
-    joint_xyz="0.0 -0.492 0.272"
+    joint_xyz="0.465 0 0.272"
     joint_rpy="0 0 0"
     mesh_xyz="0 0 0"
@@ -37,6 +37,6 @@
     name="camera"
     parent_link="base_link"
-    joint_xyz="0.0 -0.47 0.216"
-    joint_rpy="0 0 0"
+    joint_xyz="0.47 0.0 0.216"
+    joint_rpy="0 0 1.57"
     mesh_xyz="0 0 0"
     mesh_rpy="0 0 0"/>
