Commit message: Update projct structure

File: src/polebot_amr_description/assets/urdf/mecha/base.xacro (robot description, xacro)
@@ -7,14 +7,14 @@
     <parent link="base_footprint"/>
     <child link="base_link"/>
-    <origin xyz="0 0 0" rpy="0 0 -1.57"/>
+    <origin xyz="0 0 0" rpy="0 0 0"/>
   </joint>
   <link name="chassis">
     <visual>
-      <origin xyz="0 0 0" rpy="0 0 1.57"/>
-      <geometry>
-        <mesh filename="file://${mesh_path}/polebot_amr.stl" scale="0.001 0.001 0.001"/>
+      <origin xyz="0 0 0" rpy="0 0 0"/>
+      <geometry>
+        <mesh filename="package://polebot_amr_description/meshes/polebot_amr.stl" scale="0.001 0.001 0.001"/>
       </geometry>
       <material name="gray">
-        <color rgba="0.3 0.3 0.3 1.0"/>
+        <color rgba="0.5 0.5 0.5 1.0"/>
       </material>
     </visual>
@@ -64,5 +64,5 @@
     <parent link="base_link"/>
     <child link="left_wheel"/>
-    <origin xyz="0.375 0.3 0.07" rpy="1.57 0 1.57"/> <!-- Position à adapter -->
+    <origin xyz="0.375 0.3 0.07" rpy="1.57 0 0"/> <!-- Position à adapter -->
     <axis xyz="0 -1 0">
         <dynamics damping="1.0" friction="0.5"/>  <!-- Ajout ici -->
@@ -96,5 +96,5 @@
     <parent link="base_link"/>
     <child link="right_wheel"/>
-    <origin xyz="-0.375 0.3 0.07" rpy="1.57 0 1.57"/> <!-- Position à adapter -->
+    <origin xyz="-0.375 0.3 0.07" rpy="1.57 0 0"/> <!-- Position à adapter -->
     <axis xyz="0 -1 0">
         <dynamics damping="1.0" friction="0.5"/>  <!-- Ajout ici -->
@@ -124,5 +124,5 @@
     <parent link="base_link"/>
     <child link="front_left_caster"/>
-    <origin xyz="0.375 -0.3 0.07" rpy="1.57 0 1.57"/> <!-- Position adaptée -->
+    <origin xyz="0.375 -0.3 0.07" rpy="1.57 0 0"/> <!-- Position adaptée -->
     <axis xyz="0 -1 0"/>
   </joint>
@@ -150,5 +150,57 @@
     <parent link="base_link"/>
     <child link="front_right_caster"/>
-    <origin xyz="-0.375 -0.3 0.07" rpy="1.57 0 1.57"/> <!-- Position adaptée -->
+    <origin xyz="-0.375 -0.3 0.07" rpy="1.57 0 0"/> <!-- Position adaptée -->
+    <axis xyz="0 -1 0"/>
+  </joint>
+  <link name="rear_left_caster">
+    <inertial>
+      <mass value="1.5"/>
+      <inertia ixx="0.41" ixy="0" ixz="0" iyy="0.755" iyz="0" izz="0.755"/>
+    </inertial>
+    <collision>
+      <geometry>
+        <cylinder radius="0.07" length="0.05"/>
+      </geometry>
+      <origin xyz="0 0 0" rpy="0 0 0"/>
+      <surface>
+        <friction>
+          <ode>
+            <mu>1.0</mu>
+            <mu2>0.0</mu2>
+          </ode>
+        </friction>
+      </surface>
+    </collision>
+  </link>
+  <joint name="rear_left_caster_joint" type="continuous">
+    <parent link="base_link"/>
+    <child link="front_left_caster"/>
+    <origin xyz="0.375 -0.3 0.07" rpy="1.57 0 0"/> <!-- Position adaptée -->
+    <axis xyz="0 -1 0"/>
+  </joint>
+  <link name="rear_right_caster">
+    <inertial>
+      <mass value="1.5"/>
+      <inertia ixx="0.41" ixy="0" ixz="0" iyy="0.755" iyz="0" izz="0.755"/>
+    </inertial>
+    <collision>
+      <geometry>
+        <cylinder radius="0.07" length="0.05"/>
+      </geometry>
+      <origin xyz="0 0 0" rpy="0 0 0"/>
+      <surface>
+        <friction>
+          <ode>
+            <mu>1.0</mu>
+            <mu2>0.0</mu2>
+          </ode>
+        </friction>
+      </surface>
+    </collision>
+  </link>
+  <joint name="rear_right_caster_joint" type="continuous">
+    <parent link="base_link"/>
+    <child link="front_right_caster"/>
+    <origin xyz="-0.375 -0.3 0.07" rpy="1.57 0 0"/> <!-- Position adaptée -->
     <axis xyz="0 -1 0"/>
   </joint>

File: src/polebot_amr_description/assets/urdf/mecha/wheel.xacro (robot description, xacro)
@@ -17,5 +17,5 @@
         <origin xyz="0 0 0" rpy="0 0 0"/>
         <geometry>
-          <mesh filename="file://${mesh_path}/wheel.stl" scale="0.001 0.001 0.001"/>
+          <mesh filename="package://polebot_amr_description/meshes/wheel.stl" scale="0.001 0.001 0.001"/>
         </geometry>
         <material name="${name}_material">
@@ -27,5 +27,5 @@
         <origin xyz="0 0 0" rpy="0 0 0"/>
         <geometry>
-          <mesh filename="file://${mesh_path}/wheel.stl" scale="0.001 0.001 0.001"/>
+          <mesh filename="package://polebot_amr_description/meshes/wheel.stl" scale="0.001 0.001 0.001"/>
         </geometry>
       </collision>

File: src/polebot_amr_description/assets/urdf/sensors/camera.xacro (robot description, xacro)
@@ -2,5 +2,4 @@
 <robot xmlns:xacro="http://www.ros.org/wiki/xacro" name="camera">
   <xacro:property name="mesh_path" value="$(find polebot_amr_description)/meshes"/>
-  <!-- Macro pour une caméra avec pose mesh configurable -->
   <xacro:macro name="camera_sensor" params="
     name
@@ -17,5 +16,5 @@
         <origin xyz="${mesh_xyz}" rpy="${mesh_rpy}"/>
         <geometry>
-          <mesh filename="file://${mesh_path}/camera.stl" scale="0.001 0.001 0.001"/>
+          <mesh filename="package://polebot_amr_description/meshes/camera.stl" scale="0.001 0.001 0.001"/>
         </geometry>
         <material name="${name}_material">
@@ -26,5 +25,5 @@
         <origin xyz="${mesh_xyz}" rpy="${mesh_rpy}"/>
         <geometry>
-          <mesh filename="file://${mesh_path}/camera.stl" scale="0.001 0.001 0.001"/>
+          <mesh filename="package://polebot_amr_description/meshes/camera.stl" scale="0.001 0.001 0.001"/>
         </geometry>
       </collision>

File: src/polebot_amr_description/assets/urdf/sensors/lidar.xacro (robot description, xacro)
@@ -2,5 +2,4 @@
 <robot xmlns:xacro="http://www.ros.org/wiki/xacro" name="lidar">
   <xacro:property name="mesh_path" value="$(find polebot_amr_description)/meshes"/>
-  <!-- Macro lidar avec visual et collision identiques -->
   <xacro:macro name="lidar_sensor" params="
     name
@@ -8,5 +7,4 @@
     joint_xyz joint_rpy
     mesh_xyz mesh_rpy
-    mesh
     update_rate:=10
     ray_count:=270
@@ -30,8 +28,8 @@
         <origin xyz="${mesh_xyz}" rpy="${mesh_rpy}"/>
         <geometry>
-          <mesh filename="file://${mesh_path}/${mesh}" scale="0.001 0.001 0.001"/>
+          <mesh filename="package://polebot_amr_description/meshes/lidar.stl" scale="0.001 0.001 0.001"/>
         </geometry>
         <material name="${name}_material">
-          <color rgba="0.301961 0.290196 0.262745 1.0"/>
+          <color rgba="0.2 0.2 0.2 1.0"/>
         </material>
       </visual>
@@ -40,5 +38,5 @@
         <origin xyz="${mesh_xyz}" rpy="${mesh_rpy}"/>
         <geometry>
-          <mesh filename="file://${mesh_path}/${mesh}" scale="0.001 0.001 0.001"/>
+          <mesh filename="package://polebot_amr_description/meshes/lidar.stl" scale="0.001 0.001 0.001"/>
         </geometry>
       </collision>

File: src/polebot_amr_description/assets/urdf/sensors/ultrasonic.xacro (robot description, xacro)
@@ -1,6 +1,5 @@
 <?xml version="1.0"?>
-<robot xmlns:xacro="http://www.ros.org/wiki/xacro" name="ultrasonic_sensors">
+<robot xmlns:xacro="http://www.ros.org/wiki/xacro" name="ultrasonic">
   <xacro:property name="mesh_path" value="$(find polebot_amr_description)/meshes"/>
-  <!-- Macro Xacro pour un capteur ultrasonique avec position locale -->
   <xacro:macro name="ultrasonic_sensor" params="
     name
@@ -27,5 +26,5 @@
         <origin xyz="0 0 0" rpy="0 0 0"/>
         <geometry>
-          <mesh filename="file://${mesh_path}/hcsr04.stl" scale="0.001 0.001 0.001"/>
+          <mesh filename="package://polebot_amr_description/meshes/hcsr04.stl" scale="0.001 0.001 0.001"/>
         </geometry>
         <material name="${name}_material">
@@ -37,5 +36,5 @@
         <origin xyz="0 0 0" rpy="0 0 0"/>
         <geometry>
-          <mesh filename="file://${mesh_path}/hcsr04.stl" scale="0.001 0.001 0.001"/>
+          <mesh filename="package://polebot_amr_description/meshes/hcsr04.stl" scale="0.001 0.001 0.001"/>
         </geometry>
       </collision>

Commit message: Update Fix Bug for Robot Description

File: src/polebot_amr_description/assets/urdf/mecha/base.xacro (robot description, xacro)
@@ -27,6 +27,5 @@
     <inertial>
       <origin xyz="0 0 0.35" rpy="0 0 0"/>
-      <mass value="5.0"/> <!-- Poids réduit pour répartir avec roues -->
-      <!-- Inertie recalculée de manière approximative -->
+      <mass value="5.0"/>
       <inertia ixx="0.41" ixy="0" ixz="0" iyy="0.755" iyz="0" izz="0.755"/>
     </inertial>
@@ -64,5 +63,5 @@
     <parent link="base_link"/>
     <child link="left_wheel"/>
-    <origin xyz="0.375 0.3 0.07" rpy="1.57 0 0"/> <!-- Position à adapter -->
+    <origin xyz="0.0 0.3 0.07" rpy="0 0 0"/> <!-- Position à adapter -->
     <axis xyz="0 -1 0">
         <dynamics damping="1.0" friction="0.5"/>  <!-- Ajout ici -->
@@ -96,5 +95,5 @@
     <parent link="base_link"/>
     <child link="right_wheel"/>
-    <origin xyz="-0.375 0.3 0.07" rpy="1.57 0 0"/> <!-- Position à adapter -->
+    <origin xyz="0.0 -0.3 0.07" rpy="0 0 0"/> <!-- Position à adapter -->
     <axis xyz="0 -1 0">
         <dynamics damping="1.0" friction="0.5"/>  <!-- Ajout ici -->
@@ -124,5 +123,5 @@
     <parent link="base_link"/>
     <child link="front_left_caster"/>
-    <origin xyz="0.375 -0.3 0.07" rpy="1.57 0 0"/> <!-- Position adaptée -->
+    <origin xyz="0.375 0.3 0.07" rpy="0 0 0"/> <!-- Position adaptée -->
     <axis xyz="0 -1 0"/>
   </joint>
@@ -150,5 +149,5 @@
     <parent link="base_link"/>
     <child link="front_right_caster"/>
-    <origin xyz="-0.375 -0.3 0.07" rpy="1.57 0 0"/> <!-- Position adaptée -->
+    <origin xyz="0.375 -0.3 0.07" rpy="0 0 0"/> <!-- Position adaptée -->
     <axis xyz="0 -1 0"/>
   </joint>
@@ -175,6 +174,6 @@
   <joint name="rear_left_caster_joint" type="continuous">
     <parent link="base_link"/>
-    <child link="front_left_caster"/>
-    <origin xyz="0.375 -0.3 0.07" rpy="1.57 0 0"/> <!-- Position adaptée -->
+    <child link="rear_left_caster"/>
+    <origin xyz="-0.375 0.3 0.07" rpy="0 0 0"/> <!-- Position adaptée -->
     <axis xyz="0 -1 0"/>
   </joint>
@@ -201,6 +200,6 @@
   <joint name="rear_right_caster_joint" type="continuous">
     <parent link="base_link"/>
-    <child link="front_right_caster"/>
-    <origin xyz="-0.375 -0.3 0.07" rpy="1.57 0 0"/> <!-- Position adaptée -->
+    <child link="rear_right_caster"/>
+    <origin xyz="-0.375 -0.3 0.07" rpy="0 0 0"/> <!-- Position adaptée -->
     <axis xyz="0 -1 0"/>
   </joint>

File: src/polebot_amr_description/assets/urdf/robot/polebot_amr.xacro (robot description, xacro)
@@ -2,6 +2,6 @@
 <robot xmlns:xacro="http://www.ros.org/wiki/xacro" xmlns:gz="http://gazebosim.org" name="polebot_amr">
   <xacro:arg name="package_path" default="" />
-  <xacro:property name="mecha_path" value="$(arg package_path)/mecha"/>
-  <xacro:property name="sensor_path" value="$(arg package_path)/sensors"/>
+  <xacro:property name="mecha_path" value="$(arg package_path)/urdf/mecha"/>
+  <xacro:property name="sensor_path" value="$(arg package_path)/urdf/sensors"/>
   <xacro:include filename="$(arg package_path)/urdf/mecha/base.xacro"/>
   <xacro:include filename="$(arg package_path)/urdf/mecha/wheel.xacro"/>

Commit message: Update gazebo simulation package

File: src/polebot_amr_description/assets/urdf/mecha/base.xacro (robot description, xacro)
@@ -22,10 +22,10 @@
       <origin xyz="0 0 0" rpy="0 0 0"/>
       <geometry>
-        <box size="0.7 1.15 0.7"/>
-      </geometry>
-    </collision>
-    <inertial>
-      <origin xyz="0 0 0.35" rpy="0 0 0"/>
-      <mass value="5.0"/>
+        <mesh filename="package://polebot_amr_description/meshes/polebot_amr.stl" scale="0.001 0.001 0.001"/>
+      </geometry>
+    </collision>
+    <inertial>
+      <origin xyz="0 0 0" rpy="0 0 0"/>
+      <mass value="50.0"/>
       <inertia ixx="0.41" ixy="0" ixz="0" iyy="0.755" iyz="0" izz="0.755"/>
     </inertial>
@@ -37,65 +37,77 @@
   </joint>
   <link name="left_wheel">
-    <inertial>
-      <origin xyz="0 0 0" rpy="0 0 0"/>
-      <mass value="1.5"/> <!-- ↖ Plus lourd -->
-      <inertia
-        ixx="0.003" ixy="0.0" ixz="0.0"
-        iyy="0.003" iyz="0.0"
-        izz="0.002"/>
-    </inertial>
-    <collision>
-      <geometry>
-        <cylinder radius="0.07" length="0.05"/>
-      </geometry>
-      <origin xyz="0 0 0" rpy="0 0 0"/>
-      <surface>
-        <friction>
-          <ode>
-            <mu>1.0</mu>
-            <mu2>0.0</mu2>
-          </ode>
-        </friction>
-      </surface>
-    </collision>
+    <visual>
+      <origin xyz="0 0 0" rpy="0 0 0"/>
+      <geometry>
+        <mesh filename="package://polebot_amr_description/meshes/wheel.stl" scale="0.001 0.001 0.001"/>
+      </geometry>
+      <material name="gray">
+        <color rgba="0.5 0.5 0.5 1.0"/>
+      </material>
+    </visual>
+    <collision>
+      <origin xyz="0 0 0" rpy="0 0 0"/>
+      <geometry>
+        <mesh filename="package://polebot_amr_description/meshes/wheel.stl" scale="0.001 0.001 0.001"/>
+      </geometry>
+    </collision>
+    <inertial>
+      <origin xyz="0 0 0" rpy="0 0 0"/>
+      <mass value="1.5"/>
+      <inertia ixx="0.003" ixy="0" ixz="0" iyy="0.003" iyz="0" izz="0.002"/>
+      <surface>
+        <friction>
+          <ode>
+            <mu>1.0</mu>
+            <mu2>0.0</mu2>
+          </ode>
+        </friction>
+      </surface>
+    </inertial>
   </link>
   <joint name="left_wheel_joint" type="continuous">
     <parent link="base_link"/>
     <child link="left_wheel"/>
-    <origin xyz="0.0 0.3 0.07" rpy="0 0 0"/> <!-- Position à adapter -->
+    <origin xyz="0.083 0.32 0.078" rpy="0 0 0"/>
     <axis xyz="0 -1 0">
-        <dynamics damping="1.0" friction="0.5"/>  <!-- Ajout ici -->
+      <dynamics damping="1.0" friction="0.5"/>
     </axis>
   </joint>
    <link name="right_wheel">
-    <inertial>
-      <origin xyz="0 0 0" rpy="0 0 0"/>
-      <mass value="1.5"/> <!-- ↖ Plus lourd -->
-      <inertia
-        ixx="0.003" ixy="0.0" ixz="0.0"
-        iyy="0.003" iyz="0.0"
-        izz="0.002"/>
-    </inertial>
-    <collision>
-      <geometry>
-        <cylinder radius="0.07" length="0.05"/>
-      </geometry>
-      <origin xyz="0 0 0" rpy="0 0 0"/>
-      <surface>
-        <friction>
-          <ode>
-            <mu>1.0</mu>
-            <mu2>0.0</mu2>
-          </ode>
-        </friction>
-      </surface>
-    </collision>
+    <visual>
+      <origin xyz="0 0 0" rpy="0 0 3.14"/>
+      <geometry>
+        <mesh filename="package://polebot_amr_description/meshes/wheel.stl" scale="0.001 0.001 0.001"/>
+      </geometry>
+      <material name="gray">
+        <color rgba="0.5 0.5 0.5 1.0"/>
+      </material>
+    </visual>
+    <collision>
+      <origin xyz="0 0 0" rpy="0 0 3.14"/>
+      <geometry>
+        <mesh filename="package://polebot_amr_description/meshes/wheel.stl" scale="0.001 0.001 0.001"/>
+      </geometry>
+    </collision>
+    <inertial>
+      <origin xyz="0 0 0" rpy="0 0 0"/>
+      <mass value="1.5"/>
+      <inertia ixx="0.003" ixy="0" ixz="0" iyy="0.003" iyz="0" izz="0.002"/>
+      <surface>
+        <friction>
+          <ode>
+            <mu>1.0</mu>
+            <mu2>0.0</mu2>
+          </ode>
+        </friction>
+      </surface>
+    </inertial>
   </link>
   <joint name="right_wheel_joint" type="continuous">
     <parent link="base_link"/>
     <child link="right_wheel"/>
-    <origin xyz="0.0 -0.3 0.07" rpy="0 0 0"/> <!-- Position à adapter -->
+    <origin xyz="0.083 -0.32 0.078" rpy="0 0 0"/>
     <axis xyz="0 -1 0">
-        <dynamics damping="1.0" friction="0.5"/>  <!-- Ajout ici -->
+        <dynamics damping="1.0" friction="0.5"/>
     </axis>
   </joint>
@@ -107,7 +119,7 @@
     <collision>
       <geometry>
-        <cylinder radius="0.07" length="0.05"/>
-      </geometry>
-      <origin xyz="0 0 0" rpy="0 0 0"/>
+        <cylinder radius="0.06" length="0.03"/>
+      </geometry>
+      <origin xyz="0 0 0" rpy="1.57 0 0"/>
       <surface>
         <friction>
@@ -123,5 +135,5 @@
     <parent link="base_link"/>
     <child link="front_left_caster"/>
-    <origin xyz="0.375 0.3 0.07" rpy="0 0 0"/> <!-- Position adaptée -->
+    <origin xyz="0.417 0.32 0.06" rpy="0 0 0"/>
     <axis xyz="0 -1 0"/>
   </joint>
@@ -133,7 +145,7 @@
     <collision>
       <geometry>
-        <cylinder radius="0.07" length="0.05"/>
-      </geometry>
-      <origin xyz="0 0 0" rpy="0 0 0"/>
+        <cylinder radius="0.06" length="0.03"/>
+      </geometry>
+      <origin xyz="0 0 0" rpy="1.57 0 0"/>
       <surface>
         <friction>
@@ -149,5 +161,5 @@
     <parent link="base_link"/>
     <child link="front_right_caster"/>
-    <origin xyz="0.375 -0.3 0.07" rpy="0 0 0"/> <!-- Position adaptée -->
+    <origin xyz="0.417 -0.32 0.06" rpy="0 0 0"/>
     <axis xyz="0 -1 0"/>
   </joint>
@@ -159,7 +171,7 @@
     <collision>
       <geometry>
-        <cylinder radius="0.07" length="0.05"/>
-      </geometry>
-      <origin xyz="0 0 0" rpy="0 0 0"/>
+        <cylinder radius="0.06" length="0.03"/>
+      </geometry>
+      <origin xyz="0 0 0" rpy="1.57 0 0"/>
       <surface>
         <friction>
@@ -175,5 +187,5 @@
     <parent link="base_link"/>
     <child link="rear_left_caster"/>
-    <origin xyz="-0.375 0.3 0.07" rpy="0 0 0"/> <!-- Position adaptée -->
+    <origin xyz="-0.33 0.32 0.06" rpy="0 0 0"/>
     <axis xyz="0 -1 0"/>
   </joint>
@@ -185,7 +197,7 @@
     <collision>
       <geometry>
-        <cylinder radius="0.07" length="0.05"/>
-      </geometry>
-      <origin xyz="0 0 0" rpy="0 0 0"/>
+        <cylinder radius="0.06" length="0.03"/>
+      </geometry>
+      <origin xyz="0 0 0" rpy="1.57 0 0"/>
       <surface>
         <friction>
@@ -201,5 +213,5 @@
     <parent link="base_link"/>
     <child link="rear_right_caster"/>
-    <origin xyz="-0.375 -0.3 0.07" rpy="0 0 0"/> <!-- Position adaptée -->
+    <origin xyz="-0.33 -0.32 0.06" rpy="0 0 0"/>
     <axis xyz="0 -1 0"/>
   </joint>

File: src/polebot_amr_description/assets/urdf/robot/polebot_amr.xacro (robot description, xacro)
@@ -1,12 +1,9 @@
 <?xml version="1.0"?>
 <robot xmlns:xacro="http://www.ros.org/wiki/xacro" xmlns:gz="http://gazebosim.org" name="polebot_amr">
-  <xacro:arg name="package_path" default="" />
-  <xacro:property name="mecha_path" value="$(arg package_path)/urdf/mecha"/>
-  <xacro:property name="sensor_path" value="$(arg package_path)/urdf/sensors"/>
-  <xacro:include filename="$(arg package_path)/urdf/mecha/base.xacro"/>
-  <xacro:include filename="$(arg package_path)/urdf/mecha/wheel.xacro"/>
-  <xacro:include filename="$(arg package_path)/urdf/sensors/ultrasonic.xacro"/>
-  <xacro:include filename="$(arg package_path)/urdf/sensors/lidar.xacro"/>
-  <xacro:include filename="$(arg package_path)/urdf/sensors/camera.xacro"/>
+  <xacro:include filename="$(find polebot_amr_description)/urdf/mecha/base.xacro"/>
+  <xacro:include filename="$(find polebot_amr_description)/urdf/mecha/wheel.xacro"/>
+  <xacro:include filename="$(find polebot_amr_description)/urdf/sensors/ultrasonic.xacro"/>
+  <xacro:include filename="$(find polebot_amr_description)/urdf/sensors/lidar.xacro"/>
+  <xacro:include filename="$(find polebot_amr_description)/urdf/sensors/camera.xacro"/>
   <xacro:ultrasonic_sensor
     name="uls_frontleft"
@@ -32,5 +29,5 @@
     name="lidar"
     parent_link="base_link"
-    joint_xyz="0.465 0.0 0.272"
+    joint_xyz="0.470 0.0 0.272"
     joint_rpy="0 0 0"
     mesh_xyz="0 0 0"

File: src/polebot_amr_description/assets/urdf/sensors/lidar.xacro (robot description, xacro)
@@ -18,5 +18,5 @@
     visualize:=false
     enable_collision:=false">
-    <link name="${name}">
+    <link name="${name}_link">
       <inertial>
         <origin xyz="0 0 0.00977" rpy="0 0 0"/>
@@ -46,10 +46,10 @@
       <origin xyz="${joint_xyz}" rpy="${joint_rpy}"/>
       <parent link="${parent_link}"/>
-      <child link="${name}"/>
+      <child link="${name}_link"/>
       <axis xyz="0 0 1"/>
       <limit effort="10" velocity="10"/>
     </joint>
-    <gazebo reference="${name}">
-      <sensor name="lidar_sensor" type="gpu_lidar">
+    <gazebo reference="${name}_link">
+      <sensor name="lidar" type="gpu_lidar">
         <topic>${topic_name}</topic>
         <update_rate>${update_rate}</update_rate>
@@ -78,5 +78,5 @@
           </range>
         </lidar>
-        <gz_frame_id>${name}</gz_frame_id>
+        <gz_frame_id>${name}_link</gz_frame_id>
       </sensor>
     </gazebo>

File: src/polebot_amr_description/assets/urdf/sensors/ultrasonic.xacro (robot description, xacro)
@@ -16,5 +16,5 @@
     enable_collision:=false">
     <!-- Définition du lien du capteur -->
-    <link name="${name}">
+    <link name="${name}_link">
       <inertial>
         <origin xyz="0 0 0" rpy="0 0 0"/>
@@ -43,8 +43,8 @@
     <joint name="${name}_joint" type="fixed">
       <parent link="base_link"/>
-      <child link="${name}"/>
+      <child link="${name}_link"/>
       <origin xyz="${joint_xyz}" rpy="${joint_rpy}"/>
     </joint>
-    <gazebo reference="${name}">
+    <gazebo reference="${name}_link">
       <sensor name="${name}_sensor" type="gpu_lidar">
         <topic>${name}/range</topic>
@@ -67,5 +67,5 @@
           </range>
         </lidar>
-        <gz_frame_id>${name}</gz_frame_id>
+        <gz_frame_id>${name}_link</gz_frame_id>
       </sensor>
     </gazebo>
