Commit message: Debug robot description error

File: src/polebot_amr_description/assets/urdf/mecha/base.xacro (robot description, xacro)
@@ -7,5 +7,5 @@
     <parent link="base_footprint"/>
     <child link="base_link"/>
-    <origin xyz="0 0 0" rpy="0 0 0"/>
+    <origin xyz="0 0 0.180" rpy="0 0 0"/>
   </joint>
   <link name="chassis">
@@ -34,5 +34,5 @@
     <parent link="base_link"/>
     <child link="chassis"/>
-    <origin xyz="0 0 0" rpy="0 0 0"/>
+    <origin xyz="0 0 -0.180" rpy="0 0 0"/>
   </joint>
   <link name="left_wheel">
@@ -69,5 +69,5 @@
     <parent link="base_link"/>
     <child link="left_wheel"/>
-    <origin xyz="0.083 0.32 0.078" rpy="0 0 0"/>
+    <origin xyz="0.083 0.32 -0.102" rpy="0 0 0"/>
     <axis xyz="0 -1 0">
       <dynamics damping="1.0" friction="0.5"/>
@@ -107,5 +107,5 @@
     <parent link="base_link"/>
     <child link="right_wheel"/>
-    <origin xyz="0.083 -0.32 0.078" rpy="0 0 0"/>
+    <origin xyz="0.083 -0.32 -0.102" rpy="0 0 0"/>
     <axis xyz="0 -1 0">
         <dynamics damping="1.0" friction="0.5"/>
@@ -135,5 +135,5 @@
     <parent link="base_link"/>
     <child link="front_left_caster"/>
-    <origin xyz="0.417 0.32 0.06" rpy="0 0 0"/>
+    <origin xyz="0.417 0.32 -0.120" rpy="0 0 0"/>
     <axis xyz="0 -1 0"/>
   </joint>
@@ -161,5 +161,5 @@
     <parent link="base_link"/>
     <child link="front_right_caster"/>
-    <origin xyz="0.417 -0.32 0.06" rpy="0 0 0"/>
+    <origin xyz="0.417 -0.32 -0.120" rpy="0 0 0"/>
     <axis xyz="0 -1 0"/>
   </joint>
@@ -187,5 +187,5 @@
     <parent link="base_link"/>
     <child link="rear_left_caster"/>
-    <origin xyz="-0.33 0.32 0.06" rpy="0 0 0"/>
+    <origin xyz="-0.33 0.32 -0.120" rpy="0 0 0"/>
     <axis xyz="0 -1 0"/>
   </joint>
@@ -213,5 +213,5 @@
     <parent link="base_link"/>
     <child link="rear_right_caster"/>
-    <origin xyz="-0.33 -0.32 0.06" rpy="0 0 0"/>
+    <origin xyz="-0.33 -0.32 -0.120" rpy="0 0 0"/>
     <axis xyz="0 -1 0"/>
   </joint>

File: src/polebot_amr_description/assets/urdf/robot/polebot_amr.xacro (robot description, xacro)
@@ -8,20 +8,20 @@
   <xacro:ultrasonic_sensor
     name="uls_frontleft"
-    joint_xyz="0.570 0.206 0.216"
+    joint_xyz="0.570 0.206 0.06"
     joint_rpy="0 0 0"
     />
   <xacro:ultrasonic_sensor
     name="uls_frontright"
-    joint_xyz="0.570 -0.206 0.216"
+    joint_xyz="0.570 -0.206 0.06"
     joint_rpy="0 0 0"
     />
   <xacro:ultrasonic_sensor
     name="uls_backleft"
-    joint_xyz="-0.405 0.206 0.216"
+    joint_xyz="-0.405 0.206 0.06"
     joint_rpy="0 0 3.14"
     />
   <xacro:ultrasonic_sensor
     name="uls_backright"
-    joint_xyz="-0.405 -0.206 0.216"
+    joint_xyz="-0.405 -0.206 0.06"
     joint_rpy="0 0 3.14"
     />
@@ -29,6 +29,6 @@
     name="lidar"
     parent_link="base_link"
-    joint_xyz="0.470 0.0 0.272"
-    joint_rpy="0 0 0"
+    joint_xyz="0.470 0.0 0.116"
+    joint_rpy="0 0 -1.57"
     mesh_xyz="0 0 0"
     mesh_rpy="0 0 0"
@@ -37,6 +37,6 @@
     name="camera"
     parent_link="base_link"
-    joint_xyz="0.470 0.0 0.216"
-    joint_rpy="0 0 0"
+    joint_xyz="0.470 0.0 0.06"
+    joint_rpy="0 0 -1.57"
     mesh_xyz="0 0 0"
     mesh_rpy="0 0 0"

File: src/polebot_amr_description/assets/urdf/sensors/lidar.xacro (robot description, xacro)
@@ -11,8 +11,8 @@
     min_angle:='-3.1456'
     max_angle:='3.1456'
-    min_range:='0.2'
-    max_range:='30.0'
+    min_range:='0.05'
+    max_range:='25.0'
     range_resolution:='0.013'
-    topic_name:='laser_scan'
+    topic_name:='scan'
     always_on:=true
     visualize:=false
