Commit message: Debug orbbec camera integration with new robot description

File: src/polebot_amr_description/assets/urdf/robot/polebot_amr.xacro (robot description, xacro)
@@ -38,5 +38,5 @@
     parent_link="base_link"
     joint_xyz="0.470 0.0 0.06"
-    joint_rpy="0 0 -1.57"
+    joint_rpy="0 -0.09 0"
     mesh_xyz="0 0 0"
     mesh_rpy="0 0 0"

File: src/polebot_amr_description/assets/urdf/sensors/camera.xacro (robot description, xacro)
@@ -7,5 +7,5 @@
     joint_xyz joint_rpy
     mesh_xyz mesh_rpy ">
-    <link name="${name}">
+    <link name="${name}_link">
       <inertial>
         <origin xyz="0 0 0" rpy="0 0 0"/>
@@ -32,13 +32,13 @@
       <origin xyz="${joint_xyz}" rpy="${joint_rpy}"/>
       <parent link="${parent_link}"/>
-      <child link="${name}"/>
+      <child link="${name}_link"/>
     </joint>
     <joint type="fixed" name="${name}_optical_joint">
       <origin xyz="0 0 0" rpy="0 0 0"/>
-      <child link="${name}_optical"/>
-      <parent link="${name}"/>
+      <child link="${name}_link_optical"/>
+      <parent link="${name}_link"/>
     </joint>
     <!-- 6 - Camera Link Optical -->
-    <link name="${name}_optical">
+    <link name="${name}_link_optical">
     </link>
     <!-- 7 - Camera Gazebo Plugin -->
@@ -64,5 +64,5 @@
             <stddev>0.007</stddev>
           </noise>
-          <optical_frame_id>${name}_optical</optical_frame_id>
+          <optical_frame_id>${name}_link_optical</optical_frame_id>
           <camera_info_topic>${name}/camera_info</camera_info_topic>
         </camera>
