Commit message: Update robot description for slam application

File: src/polebot_amr_description/assets/urdf/sensors/camera.xacro (robot description, xacro)
@@ -7,5 +7,5 @@
     joint_xyz joint_rpy
     mesh_xyz mesh_rpy ">
-    <link name="${name}_link">
+    <link name="${name}">
       <inertial>
         <origin xyz="0 0 0" rpy="0 0 0"/>
@@ -32,16 +32,16 @@
       <origin xyz="${joint_xyz}" rpy="${joint_rpy}"/>
       <parent link="${parent_link}"/>
-      <child link="${name}_link"/>
+      <child link="${name}"/>
     </joint>
     <joint type="fixed" name="${name}_optical_joint">
       <origin xyz="0 0 0" rpy="0 0 0"/>
-      <child link="${name}_link_optical"/>
-      <parent link="${name}_link"/>
+      <child link="${name}_optical"/>
+      <parent link="${name}"/>
     </joint>
     <!-- 6 - Camera Link Optical -->
-    <link name="${name}_link_optical">
+    <link name="${name}_optical">
     </link>
     <!-- 7 - Camera Gazebo Plugin -->
-    <gazebo reference="${name}_link">
+    <gazebo reference="${name}">
       <sensor name="${name}" type="camera">
         <camera>
@@ -64,5 +64,5 @@
             <stddev>0.007</stddev>
           </noise>
-          <optical_frame_id>${name}_link_optical</optical_frame_id>
+          <optical_frame_id>${name}_optical</optical_frame_id>
           <camera_info_topic>${name}/camera_info</camera_info_topic>
         </camera>

Commit message: Debug robot simulation with gazebo

File: src/polebot_amr_description/assets/urdf/sensors/camera.xacro (robot description, xacro)
@@ -1,13 +1,12 @@
 <?xml version="1.0"?>
 <robot xmlns:xacro="http://www.ros.org/wiki/xacro" name="camera">
-  <xacro:property name="mesh_path" value="$(find polebot_amr_description)/meshes"/>
   <xacro:macro name="camera_sensor" params="
     name
     parent_link
     joint_xyz joint_rpy
-    mesh_xyz mesh_rpy ">
+    mesh_xyz:='0 0 0' mesh_rpy:='0 0 0'">
+    <!-- Main camera link -->
     <link name="${name}_link">
       <inertial>
-        <origin xyz="0 0 0" rpy="0 0 0"/>
         <mass value="0.1"/>
         <inertia ixx="1e-05" ixy="0" ixz="0" iyy="1e-05" iyz="0" izz="1e-05"/>
@@ -23,26 +22,27 @@
       </visual>
       <collision>
-        <origin xyz="${mesh_xyz}" rpy="${mesh_rpy}"/>
         <geometry>
-          <mesh filename="package://polebot_amr_description/meshes/camera.stl" scale="0.001 0.001 0.001"/>
+          <box size="0.02 0.03 0.01"/>
         </geometry>
       </collision>
     </link>
+    <!-- Fixed joint to robot -->
     <joint name="${name}_joint" type="fixed">
-      <origin xyz="${joint_xyz}" rpy="${joint_rpy}"/>
       <parent link="${parent_link}"/>
       <child link="${name}_link"/>
+      <origin xyz="${joint_xyz}" rpy="${joint_rpy}"/>
     </joint>
-    <joint type="fixed" name="${name}_optical_joint">
-      <origin xyz="0 0 0" rpy="0 0 0"/>
+    <!-- Optical frame (Z forward, X right, Y down) -->
+    <link name="${name}_link_optical"/>
+    <joint name="${name}_optical_joint" type="fixed">
+      <parent link="${name}_link"/>
       <child link="${name}_link_optical"/>
-      <parent link="${name}_link"/>
+      <origin xyz="0 0 0" rpy="-1.5708 0 -1.5708"/> <!-- 90° around X and Z -->
     </joint>
-    <!-- 6 - Camera Link Optical -->
-    <link name="${name}_link_optical">
-    </link>
-    <!-- 7 - Camera Gazebo Plugin -->
-    <gazebo reference="${name}">
+    <!-- Gazebo camera sensor (OUTSIDE link) -->
+    <gazebo reference="${name}_link">
       <sensor name="${name}" type="camera">
+        <topic>/camera/image</topic>
+        <update_rate>30</update_rate>
         <camera>
           <horizontal_fov>1.1</horizontal_fov>
@@ -54,21 +54,14 @@
           <clip>
             <near>0.1</near>
-            <far>15</far>
+            <far>15.0</far>
           </clip>
-          <noise>
-            <type>gaussian</type>
-            <!-- Noise is sampled independently per pixel on each frame.
-                That pixel's noise value is added to each of its color
-                channels, which at that point lie in the range [0,1]. -->
-            <mean>0.0</mean>
-            <stddev>0.007</stddev>
-          </noise>
-          <optical_frame_id>${name}_link_optical</optical_frame_id>
-          <camera_info_topic>${name}/camera_info</camera_info_topic>
         </camera>
-        <always_on>1</always_on>
-        <update_rate>20</update_rate>
-        <visualize>true</visualize>
-        <topic>${name}/image</topic>
+        <plugin filename="libros_gz_sensor_plugin.so" name="ros_gz::SensorPlugin">
+          <ros>
+            <frame_id>${name}_link_optical</frame_id>
+            <remapping>/camera/image:=/camera/image_raw</remapping>
+            <remapping>/camera/camera_info:=/camera/camera_info</remapping>
+          </ros>
+        </plugin>
       </sensor>
     </gazebo>

File: src/polebot_amr_description/assets/urdf/sensors/lidar.xacro (robot description, xacro)
@@ -9,6 +9,6 @@
     update_rate:=10
     ray_count:=270
-    min_angle:='-3.1456'
-    max_angle:='3.1456'
+    min_angle:='-2.3592'
+    max_angle:='2.3592'
     min_range:='0.05'
     max_range:='25.0'
@@ -16,56 +16,32 @@
     topic_name:='scan'
     always_on:=true
-    visualize:=false
-    enable_collision:=false">
+    visualize:=true">
+    <!-- Link -->
     <link name="${name}_link">
-      <inertial>
-        <origin xyz="0 0 0.00977" rpy="0 0 0"/>
-        <mass value="0.02915"/>
-        <inertia ixx="3.79e-06" ixy="0" ixz="0" iyy="3.79e-06" iyz="0" izz="5.71e-06"/>
-      </inertial>
-      <!-- Visual -->
-      <visual>
-        <origin xyz="${mesh_xyz}" rpy="${mesh_rpy}"/>
-        <geometry>
-          <mesh filename="package://polebot_amr_description/meshes/lidar.stl" scale="0.001 0.001 0.001"/>
-        </geometry>
-        <material name="${name}_material">
-          <color rgba="0.2 0.2 0.2 1.0"/>
-        </material>
-      </visual>
-      <!-- Collision (identique au visual) -->
-      <collision>
-        <origin xyz="${mesh_xyz}" rpy="${mesh_rpy}"/>
-        <geometry>
-          <mesh filename="package://polebot_amr_description/meshes/lidar.stl" scale="0.001 0.001 0.001"/>
-        </geometry>
-      </collision>
+      <inertial> ... </inertial>
+      <visual> ... </visual>
+      <collision> ... </collision>
+      <!-- NO <gazebo> inside here -->
     </link>
-    <!-- Joint fixe -->
+    <!-- Joint -->
     <joint name="${name}_joint" type="fixed">
-      <origin xyz="${joint_xyz}" rpy="${joint_rpy}"/>
       <parent link="${parent_link}"/>
       <child link="${name}_link"/>
-      <axis xyz="0 0 1"/>
-      <limit effort="10" velocity="10"/>
+      <origin xyz="${joint_xyz}" rpy="${joint_rpy}"/>
     </joint>
+    <!-- Gazebo sensor (outside link!) -->
     <gazebo reference="${name}_link">
-      <sensor name="lidar" type="gpu_lidar">
-        <topic>${topic_name}</topic>
-        <update_rate>${update_rate}</update_rate>
-        <always_on>${always_on}</always_on>
-        <visualize>${visualize}</visualize>
+      <sensor name="${name}" type="gpu_lidar">
+        <topic>${name}/scan</topic>
+        <update_rate>10</update_rate>
         <lidar>
           <scan>
             <horizontal>
-              <samples>${ray_count}</samples>
-              <resolution>1</resolution>
-              <min_angle>${min_angle}</min_angle>
-              <max_angle>${max_angle}</max_angle>
+              <samples>270</samples>
+              <min_angle>-3.14</min_angle>
+              <max_angle>3.14</max_angle>
             </horizontal>
-            <!-- 2D Lidar -->
             <vertical>
               <samples>1</samples>
-              <resolution>1</resolution>
               <min_angle>0</min_angle>
               <max_angle>0</max_angle>
@@ -73,10 +49,14 @@
           </scan>
           <range>
-            <min>${min_range}</min>
-            <max>${max_range}</max>
-            <resolution>${range_resolution}</resolution>
+            <min>0.05</min>
+            <max>25.0</max>
           </range>
         </lidar>
-        <gz_frame_id>${name}_link</gz_frame_id>
+        <plugin filename="libros_gz_sensor_plugin.so" name="ros_gz::SensorPlugin">
+          <ros>
+            <frame_id>${name}_link</frame_id>
+            <remapping>${name}/scan:=/scan</remapping>
+          </ros>
+        </plugin>
       </sensor>
     </gazebo>

File: src/polebot_amr_description/assets/urdf/sensors/ultrasonic.xacro (robot description, xacro)
@@ -1,28 +1,20 @@
 <?xml version="1.0"?>
 <robot xmlns:xacro="http://www.ros.org/wiki/xacro" name="ultrasonic">
-  <xacro:property name="mesh_path" value="$(find polebot_amr_description)/meshes"/>
   <xacro:macro name="ultrasonic_sensor" params="
     name
     joint_xyz joint_rpy
-    update_rate:=10
-    ray_count:=5
-    min_angle:='-1.702'
-    max_angle:='-1.422'
     min_range:='0.02'
     max_range:='4.0'
-    range_resolution:='0.01'
+    update_rate:=10
+    fov:=0.349
     always_on:=true
-    visualize:=false
-    enable_collision:=false">
-    <!-- Définition du lien du capteur -->
+    visualize:=false">
+    <!-- Link -->
     <link name="${name}_link">
       <inertial>
-        <origin xyz="0 0 0" rpy="0 0 0"/>
         <mass value="0.0045"/>
         <inertia ixx="1e-7" ixy="0" ixz="0" iyy="5e-7" iyz="0" izz="6e-7"/>
       </inertial>
-      <!-- Visual -->
       <visual>
-        <origin xyz="0 0 0" rpy="0 0 0"/>
         <geometry>
           <mesh filename="package://polebot_amr_description/meshes/hcsr04.stl" scale="0.001 0.001 0.001"/>
@@ -32,13 +24,12 @@
         </material>
       </visual>
-      <!-- Collision -->
+      <!-- Simple collision -->
       <collision>
-        <origin xyz="0 0 0" rpy="0 0 0"/>
         <geometry>
-          <mesh filename="package://polebot_amr_description/meshes/hcsr04.stl" scale="0.001 0.001 0.001"/>
+          <cylinder radius="0.01" length="0.02"/>
         </geometry>
       </collision>
     </link>
-    <!-- Joint fixe entre le capteur et le parent -->
+    <!-- Fixed joint -->
     <joint name="${name}_joint" type="fixed">
       <parent link="base_link"/>
@@ -46,7 +37,8 @@
       <origin xyz="${joint_xyz}" rpy="${joint_rpy}"/>
     </joint>
+    <!-- Gazebo: 1-beam ray sensor (ultrasonic approximation) -->
     <gazebo reference="${name}_link">
-      <sensor name="${name}_sensor" type="gpu_lidar">
-        <topic>${name}/range</topic>
+      <sensor name="${name}" type="gpu_lidar">
+        <topic>/ultrasonic/${name}</topic>
         <update_rate>${update_rate}</update_rate>
         <always_on>${always_on}</always_on>
@@ -55,17 +47,24 @@
           <scan>
             <horizontal>
-              <samples>${ray_count}</samples>
-              <resolution>1</resolution>
-              <min_angle>${min_angle}</min_angle>
-              <max_angle>${max_angle}</max_angle>
+              <samples>1</samples>              <!-- ONLY 1 BEAM -->
+              <min_angle>0</min_angle>          <!-- CENTERED -->
+              <max_angle>0</max_angle>
             </horizontal>
+            <vertical>
+              <samples>1</samples>
+              <min_angle>0</min_angle>
+              <max_angle>0</max_angle>
+            </vertical>
           </scan>
           <range>
             <min>${min_range}</min>
             <max>${max_range}</max>
-            <resolution>${range_resolution}</resolution>
           </range>
         </lidar>
-        <gz_frame_id>${name}_link</gz_frame_id>
+        <plugin filename="libros_gz_sensor_plugin.so" name="ros_gz::SensorPlugin">
+          <ros>
+            <frame_id>${name}_link</frame_id>
+          </ros>
+        </plugin>
       </sensor>
     </gazebo>
